File: esp32.kicad_sch (KiCad schematic)
At the start: 21 parts, among them J2 TC2030-IDC, J3 Conn_01x04, J4 Conn_01x06, J5 USB_C_Receptacle_USB2.0, SW1 GT-TC029B-H025-L1N, SW2 GT-TC029B-H025-L1N, U3 RT9080-33GJ5, U4 ESP32-S3-WROOM-1

Commit message: Add BitcoinMerch Logo
Changed lines of the file:
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@@
 (kicad_sch
-	(version 20231120)
+	(version 20250114)
 	(generator "eeschema")
-	(generator_version "8.0")
+	(generator_version "9.0")
 	(paper "A")
 	(title_block
@@
 		(rev "402")
 	)
+	(text "Accessory Port"
+		(exclude_from_sim no)
+		(at 220.98 113.03 0)
+		(effects
+			(font
+				(size 1.27 1.27)
+			)
+			(justify left bottom)
+		)
+	)
+	(text "ESP32 3V3 LDO"
+		(exclude_from_sim no)
+		(at 41.91 45.72 0)
+		(effects
+			(font
+				(size 1.27 1.27)
+			)
+			(justify left bottom)
+		)
+	)
+	(text "Program the ESP32 with a ESP-PROG and a Tag Connect TC2030-IDC"
+		(exclude_from_sim no)
+		(at 30.353 179.451 0)
+		(effects
+			(font
+				(size 1.27 1.27)
+			)
+			(justify left bottom)
+		)
+	)
+	(text "SSD1306 128x32 I2C OLED"
+		(exclude_from_sim no)
+		(at 186.182 44.958 0)
+		(effects
+			(font
+				(size 1.27 1.27)
+			)
+			(justify left bottom)
+		)
+	)
+	(text "OLED Display Header"
+		(exclude_from_sim no)
+		(at 188.722 41.783 0)
+		(effects
+			(font
+				(size 1.27 1.27)
+			)
+			(justify left bottom)
+		)
+	)
 	(junction
 		(at 214.63 69.215)
@@
 		)
 	)
-	(text "Accessory Port"
-		(exclude_from_sim no)
-		(at 220.98 113.03 0)
-		(effects
-			(font
-				(size 1.27 1.27)
-			)
-			(justify left bottom)
-		)
-	)
-	(text "ESP32 3V3 LDO"
-		(exclude_from_sim no)
-		(at 41.91 45.72 0)
-		(effects
-			(font
-				(size 1.27 1.27)
-			)
-			(justify left bottom)
-		)
-	)
-	(text "Program the ESP32 with a ESP-PROG and a Tag Connect TC2030-IDC"
-		(exclude_from_sim no)
-		(at 30.353 179.451 0)
-		(effects
-			(font
-				(size 1.27 1.27)
-			)
-			(justify left bottom)
-		)
-	)
-	(text "SSD1306 128x32 I2C OLED"
-		(exclude_from_sim no)
-		(at 186.182 44.958 0)
-		(effects
-			(font
-				(size 1.27 1.27)
-			)
-			(justify left bottom)
-		)
-	)
-	(text "OLED Display Header"
-		(exclude_from_sim no)
-		(at 188.722 41.783 0)
-		(effects
-			(font
-				(size 1.27 1.27)
-			)
-			(justify left bottom)
-		)
-	)
 	(label "P_RX"
 		(at 52.07 171.45 0)
-		(fields_autoplaced yes)
 		(effects
 			(font
@@
 	(label "RST"
 		(at 69.85 85.09 0)
-		(fields_autoplaced yes)
 		(effects
 			(font
@@
 	(label "P_TX"
 		(at 52.07 168.91 0)
-		(fields_autoplaced yes)
 		(effects
 			(font
@@
 	(label "EN"
 		(at 52.07 166.37 0)
-		(fields_autoplaced yes)
 		(effects
 			(font
@@
 	(label "GND"
 		(at 184.912 29.845 0)
-		(fields_autoplaced yes)
 		(effects
 			(font
@@
 	(label "5V"
 		(at 213.36 115.57 0)
-		(fields_autoplaced yes)
 		(effects
 			(font
@@
 	(label "GND"
 		(at 224.79 92.075 0)
-		(fields_autoplaced yes)
 		(effects
 			(font
@@
 	(label "EN"
 		(at 68.58 80.01 0)
-		(fields_autoplaced yes)
 		(effects
 			(font
@@
 	(label "P_RX"
 		(at 195.58 90.17 0)
-		(fields_autoplaced yes)
 		(effects
 			(font
@@
 	(label "IO0"
 		(at 68.58 77.47 0)
-		(fields_autoplaced yes)
 		(effects
 			(font
@@
 	(label "GND"
 		(at 125.73 68.58 0)
-		(fields_autoplaced yes)
 		(effects
 			(font
@@
 	(label "3V3"
 		(at 66.675 135.89 0)
-		(fields_autoplaced yes)
 		(effects
 			(font
@@
 	(label "USB_D-"
 		(at 203.2 80.01 0)
-		(fields_autoplaced yes)
 		(effects
 			(font
@@
 	(label "SDA"
 		(at 195.58 102.87 0)
-		(fields_autoplaced yes)
 		(effects
 			(font
@@
 	(label "TX"
 		(at 70.485 125.73 0)
-		(fields_autoplaced yes)
 		(effects
 			(font
@@
 	(label "3V3"
 		(at 77.47 166.37 0)
-		(fields_autoplaced yes)
 		(effects
 			(font
@@
 	(label "3V3"
 		(at 69.85 90.17 0)
-		(fields_autoplaced yes)
 		(effects
 			(font
@@
 	(label "IO0"
 		(at 77.47 171.45 0)
-		(fields_autoplaced yes)
 		(effects
 			(font
@@
 	(label "SCL"
 		(at 195.58 100.33 0)
-		(fields_autoplaced yes)
 		(effects
 			(font
@@
 	(label "SCL"
 		(at 184.912 34.925 0)
-		(fields_autoplaced yes)
 		(effects
 			(font
@@
 	(label "GND"
 		(at 213.36 118.11 0)
-		(fields_autoplaced yes)
 		(effects
 			(font
@@
 	(label "GND"
 		(at 201.93 135.89 0)
-		(fields_autoplaced yes)
 		(effects
 			(font
@@
 	(label "GND"
 		(at 45.72 77.47 0)
-		(fields_autoplaced yes)
 		(effects
 			(font
@@
 	(label "SDA"
 		(at 184.912 37.465 0)
-		(fields_autoplaced yes)
 		(effects
 			(font
@@
 	(label "3V3"
 		(at 125.73 55.88 0)
-		(fields_autoplaced yes)
 		(effects
 			(font
@@
 	(label "P_TX"
 		(at 195.58 87.63 0)
-		(fields_autoplaced yes)
 		(effects
 			(font
@@
 	(label "3V3"
 		(at 184.912 32.385 0)
-		(fields_autoplaced yes)
 		(effects
 			(font
@@
 	(label "GND"
 		(at 25.4 92.075 0)
-		(fields_autoplaced yes)
 		(effects
 			(font
@@
 	(label "5V"
 		(at 33.655 29.21 0)
-		(fields_autoplaced yes)
 		(effects
 			(font
@@
 	(label "USB_D+"
 		(at 203.2 77.47 0)
-		(fields_autoplaced yes)
 		(effects
 			(font
@@
 	(label "GND"
 		(at 77.47 168.91 0)
-		(fields_autoplaced yes)
 		(effects
 			(font
@@
 	(label "GND"
 		(at 48.895 42.545 0)
-		(fields_autoplaced yes)
 		(effects
 			(font
@@
 	(label "3V3"
 		(at 35.56 66.675 0)
-		(fields_autoplaced yes)
 		(effects
 			(font
@@
 	(label "RX"
 		(at 70.485 128.27 0)
-		(fields_autoplaced yes)
 		(effects
 			(font
@@
 		(shape input)
 		(at 66.04 125.73 180)
-		(fields_autoplaced yes)
 		(effects
 			(font
@@
 		(shape input)
 		(at 66.04 128.27 180)
-		(fields_autoplaced yes)
 		(effects
 			(font
@@
 		(shape input)
 		(at 73.025 29.21 0)
-		(fields_autoplaced yes)
 		(effects
 			(font
@@
 		(shape input)
 		(at 200.025 100.33 0)
-		(fields_autoplaced yes)
 		(effects
 			(font
@@
 		(shape input)
 		(at 66.04 85.09 180)
-		(fields_autoplaced yes)
 		(effects
 			(font
@@
 		(shape input)
 		(at 200.025 102.87 0)
-		(fields_autoplaced yes)
 		(effects
 			(font
@@
 		(shape output)
 		(at 66.04 110.49 180)
-		(fields_autoplaced yes)
 		(effects
 			(font
@@
 		(shape input)
 		(at 66.04 115.57 180)
-		(fields_autoplaced yes)
 		(effects
 			(font
@@
 		(shape input)
 		(at 23.495 29.21 180)
-		(fields_autoplaced yes)
 		(effects
 			(font
@@
 		(shape input)
 		(at 66.04 87.63 180)
-		(fields_autoplaced yes)
 		(effects
 			(font
@@
 			)
 		)
-		(property "Description" ""
+		(property "Description" "C29266"
 			(at 35.56 86.995 0)
 			(effects
@@
 			)
 		)
-		(property "Description" ""
+		(property "Description" "C159816"
 			(at 132.715 62.23 0)
 			(effects
@@
 			)
 		)
-		(property "Description" ""
+		(property "Description" "C7509546"
 			(at 196.85 32.385 0)
 			(effects
@@
 			)
 		)
-		(property "Description" ""
+		(property "Description" "C18077675"
 			(at 57.785 77.47 0)
 			(effects
@@
 			)
 		)
-		(property "Description" ""
+		(property "Description" "C841192"
 			(at 51.435 30.48 0)
 			(effects
@@
 			)
 		)
-		(property "Description" ""
+		(property "Description" "C60489"
 			(at 35.56 73.025 0)
 			(effects
@@
 			)
 		)
-		(property "Description" ""
+		(property "Description" "C29266"
 			(at 69.215 35.56 0)
 			(effects
@@
 			)
 		)
-		(property "Description" ""
+		(property "Description" "C2932476"
 			(at 121.92 62.23 0)
 			(effects
@@
 			)
 		)
-		(property "Description" ""
+		(property "Description" "C2927037"
 			(at 238.125 69.215 0)
 			(effects
@@
 			)
 		)
-		(property "Description" ""
+		(property "Description" "C29266"
 			(at 31.115 35.56 0)
 			(effects
@@
 			)
 		)
-		(property "Description" ""
+		(property "Description" "C2913202"
 			(at 133.35 107.95 0)
 			(effects
@@
 			)
 		)
-		(property "Description" ""
+		(property "Description" "C18077675"
 			(at 26.035 81.915 0)
 			(effects
