File: bm1366.kicad_sch (KiCad schematic)
At the start: 47 parts, among them U12 BM1366_mode1, U5 MCP1824T-1202E/OT, U6 MCP1824T-0802E, U7 25MHz, U9 SN74AVC4T774

Commit message: finalize
Parts:
- renumbered R6 to R17
