File: power.kicad_sch (KiCad schematic)
At the start: 40 parts, among them T1 net-tie, U2 TPS546D24ARVFR

Commit message: finalize
Parts:
- C10: PARTNO GRM155R61A475MEAAD -> CL05A475MP5NRNC
- C13: PARTNO 885012005013 -> CC0402JRNPO9BN101
- C6: PARTNO GRM155R71E472KA01D -> CC0402KRX7R8BB472
- L1: PARTNO SLC1175-301MEC -> YLSI100808-R22K
